Commit message: 日常维护

File: urdf/car_no_kinect.urdf (robot description, URDF)
Before this commit: robot differential_wheeled_robot, 7 links, 6 joints
Joints:
- joint camera_joint: origin xyz=0.125 0 0.0325 rpy=0 0 0 -> xyz=0 0 0.1 rpy=0 0 0
- joint hokuyo_joint: origin xyz=0 0 0.1 rpy=0 0 0 -> xyz=0.125 0 0.0325 rpy=0 0 0; parent camera_link -> base_link

Commit message: 移动小车摄像头

File: urdf/car_no_kinect.urdf (robot description, URDF)
Before this commit: robot differential_wheeled_robot, 7 links, 6 joints
Joints:
- joint camera_joint: origin xyz=0 0 0.1 rpy=0 0 0 -> xyz=0 0 0.1 rpy=0 0 -1.57

Commit message: 修改小车车体

File: urdf/car_no_kinect.urdf (robot description, URDF)
Before this commit: robot differential_wheeled_robot, 7 links, 6 joints
Links:
- link base_link: geometry collision box size=0.28 0.17 0.05; visual box size=0.2 0.2 0.05
Joints:
- joint back_left_wheel_joint: origin xyz=-0.10 0.095 0.0 rpy=0 0 0 -> xyz=-0.07 0.095 0.0 rpy=0 0 0
- joint back_right_wheel_joint: origin xyz=-0.10 -0.095 0.0 rpy=0 0 0 -> xyz=-0.07 -0.095 0.0 rpy=0 0 0
- joint front_left_wheel_joint: origin xyz=0.10 0.095 0.0 rpy=0 0 0 -> xyz=0.07 0.095 0.0 rpy=0 0 0
- joint front_right_wheel_joint: origin xyz=0.10 -0.095 0.0 rpy=0 0 0 -> xyz=0.07 -0.095 0.0 rpy=0 0 0
- joint hokuyo_joint: origin xyz=0.125 0 0.0325 rpy=0 0 0 -> xyz=0.065 0 0.0325 rpy=0 0 0
