Commit message: 调整小车模型参数

File: urdf/car.urdf (robot description, URDF)
Before this commit: robot differential_wheeled_robot, 6 links, 5 joints
Links:
- removed link caster_back_link
- removed link caster_front_link
- added link back_left_wheel, mass 2.5; collision cylinder length=0.03 radius=0.032; visual cylinder length=0.03 radius=0.032
- added link back_right_wheel, mass 2.5; collision cylinder length=0.03 radius=0.032; visual cylinder length=0.03 radius=0.032
- added link hokuyo_link, mass 1e-5; collision box size=.05 .05 .05; visual mesh filename=package://gx2019_omni_simulations/urdf/meshes/hokuyo.dae
- link base_link: geometry collision box size=0.28 0.17 0.05; visual box size=0.2 0.2 0.05
- link front_left_wheel: geometry collision cylinder length=0.03 radius=0.032; visual cylinder length=0.03 radius=0.032
- link front_right_wheel: geometry collision cylinder length=0.03 radius=0.032; visual cylinder length=0.03 radius=0.032
Joints:
- removed joint caster_back_joint
- removed joint caster_front_joint
- added joint back_left_wheel_joint: type continuous, parent base_link, child back_left_wheel, origin xyz=-0.07 0.095 0.0 rpy=0 0 0, axis 0 1 0, limit effort=100 velocity=100
- added joint back_right_wheel_joint: type continuous, parent base_link, child back_right_wheel, origin xyz=-0.07 -0.095 0.0 rpy=0 0 0, axis 0 1 0, limit effort=100 velocity=100
- added joint hokuyo_joint: type fixed, parent base_link, child hokuyo_link, origin xyz=0.065 0 0.0325 rpy=0 0 -3.14, axis 0 1 0
- joint camera_joint: origin xyz=0.125 0 0.0325 rpy=0 0 0 -> xyz=0 0 0.1 rpy=0 0 -1.57
- joint front_left_wheel_joint: origin xyz=0.0 -0.15 0.0 rpy=0 0 0 -> xyz=0.07 0.095 0.0 rpy=0 0 0
- joint front_right_wheel_joint: origin xyz=0.0 0.15 0.0 rpy=0 0 0 -> xyz=0.07 -0.095 0.0 rpy=0 0 0

Commit message: 添加IMU

File: urdf/car.urdf (robot description, URDF)
Before this commit: robot differential_wheeled_robot, 7 links, 6 joints
Links:
- added link imu_link; visual box size=0.05 0.05 0.05
Joints:
- added joint imu_joint: type fixed, parent base_link, child imu_joint, origin xyz=0 0 0.05 rpy=0 0 0

Commit message: imu_link_ is not correct

File: urdf/car.urdf (robot description, URDF)
Before this commit: robot differential_wheeled_robot, 8 links, 7 joints
Joints:
- joint imu_joint: child imu_joint -> imu_link

Commit message: 更新

File: urdf/car.urdf (robot description, URDF)
Before this commit: robot differential_wheeled_robot, 8 links, 7 joints
Links:
- removed link imu_link
- added link imu_link_; visual box size=0.05 0.05 0.05
Joints:
- joint imu_joint: child imu_link -> imu_link_
